File: Freezer test board/Freezer test board.kicad_sch (KiCad schematic)
At the start: 19 parts, among them J2 Conn_02x20_Odd_Even, J3 284391-3, J4 284391-3, J5 284391-3, J6 284391-3, J7 284391-3, J8 284391-3, J9 284391-3

Commit message: Finial Touches
put what specific resistors are being used in the comments. Made the finial touches and re traced the resistors and spaced them further from the terminal blocks
Parts:
- R1, R2, R3, R4, R5, R6, R7: footprint Resistor_THT:R_Axial_DIN0204_L3.6mm_D1.6mm_P5.08mm_Horizontal -> Resistor_THT:R_Axial_DIN0207_L6.3mm_D2.5mm_P7.62mm_Horizontal
Changed lines of the file:
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@@
 	(generator_version "9.0")
 	(paper "USLedger")
+	(title_block
+		(comment 1 "4.7K resistors Horizontal, pin pitch=7.62mm, 0.25W = 1/4W, ")
+	)
 	(text_box "https://www.digikey.com/en/products/detail/same-sky-formerly-cui-devices/TB007-508-03BE/10064128"
 		(exclude_from_sim no)
@@
 	)
 	(junction
-		(at 201.93 153.67)
-		(diameter 0)
-		(color 0 0 0 0)
-	)
-	(junction
 		(at 201.93 180.34)
 		(diameter 0)
@@
 	)
 	(junction
-		(at 201.93 146.05)
+		(at 201.93 153.67)
 		(diameter 0)
 		(color 0 0 0 0)
@@
 		(color 0 0 0 0)
 	)
+	(junction
+		(at 201.93 146.05)
+		(diameter 0)
+		(color 0 0 0 0)
+	)
 	(no_connect
 		(at 151.13 124.46)
@@
 	(wire
 		(pts
-			(xy 201.93 146.05) (xy 207.01 146.05)
+			(xy 198.12 77.47) (xy 201.93 77.47)
 		)
 		(stroke
@@
 	(wire
 		(pts
-			(xy 198.12 77.47) (xy 201.93 77.47)
+			(xy 201.93 54.61) (xy 198.12 54.61)
 		)
 		(stroke
@@
 	(wire
 		(pts
-			(xy 201.93 54.61) (xy 198.12 54.61)
+			(xy 201.93 123.19) (xy 207.01 123.19)
 		)
 		(stroke
@@
 	(wire
 		(pts
-			(xy 201.93 123.19) (xy 207.01 123.19)
+			(xy 201.93 153.67) (xy 207.01 153.67)
 		)
 		(stroke
@@
 	(wire
 		(pts
-			(xy 201.93 153.67) (xy 207.01 153.67)
-		)
-		(stroke
-			(width 0)
-			(type default)
-		)
-	)
-	(wire
-		(pts
 			(xy 133.35 124.46) (xy 138.43 124.46)
 		)
@@
 		)
 	)
+	(wire
+		(pts
+			(xy 201.93 146.05) (xy 207.01 146.05)
+		)
+		(stroke
+			(width 0)
+			(type default)
+		)
+	)
 	(global_label "GPIO6"
 		(shape input)
@@
 			)
 		)
-		(property "Footprint" "Resistor_THT:R_Axial_DIN0204_L3.6mm_D1.6mm_P5.08mm_Horizontal"
+		(property "Footprint" "Resistor_THT:R_Axial_DIN0207_L6.3mm_D2.5mm_P7.62mm_Horizontal"
 			(at 203.708 102.87 90)
 			(effects
@@
 			)
 		)
-		(property "Footprint" "Resistor_THT:R_Axial_DIN0204_L3.6mm_D1.6mm_P5.08mm_Horizontal"
+		(property "Footprint" "Resistor_THT:R_Axial_DIN0207_L6.3mm_D2.5mm_P7.62mm_Horizontal"
 			(at 203.708 149.86 90)
 			(effects
@@
 			)
 		)
-		(property "Footprint" "Resistor_THT:R_Axial_DIN0204_L3.6mm_D1.6mm_P5.08mm_Horizontal"
+		(property "Footprint" "Resistor_THT:R_Axial_DIN0207_L6.3mm_D2.5mm_P7.62mm_Horizontal"
 			(at 203.708 58.42 90)
 			(effects
@@
 			)
 		)
-		(property "Footprint" "Resistor_THT:R_Axial_DIN0204_L3.6mm_D1.6mm_P5.08mm_Horizontal"
+		(property "Footprint" "Resistor_THT:R_Axial_DIN0207_L6.3mm_D2.5mm_P7.62mm_Horizontal"
 			(at 203.708 81.28 90)
 			(effects
@@
 			)
 		)
-		(property "Footprint" "Resistor_THT:R_Axial_DIN0204_L3.6mm_D1.6mm_P5.08mm_Horizontal"
+		(property "Footprint" "Resistor_THT:R_Axial_DIN0207_L6.3mm_D2.5mm_P7.62mm_Horizontal"
 			(at 203.708 127 90)
 			(effects
@@
 			)
 		)
-		(property "Footprint" "Resistor_THT:R_Axial_DIN0204_L3.6mm_D1.6mm_P5.08mm_Horizontal"
+		(property "Footprint" "Resistor_THT:R_Axial_DIN0207_L6.3mm_D2.5mm_P7.62mm_Horizontal"
 			(at 203.708 200.66 90)
 			(effects
@@
 			)
 		)
-		(property "Footprint" "Resistor_THT:R_Axial_DIN0204_L3.6mm_D1.6mm_P5.08mm_Horizontal"
+		(property "Footprint" "Resistor_THT:R_Axial_DIN0207_L6.3mm_D2.5mm_P7.62mm_Horizontal"
 			(at 203.708 176.53 90)
 			(effects
