File: Freezer test board/Freezer test board.kicad_pcb (KiCad board)
At the start: 4 copper layers, 56 x 65 mm, 24 parts, among them J2 Conn_02x20_Odd_Even, J3 284391-3, J4 284391-3, J5 284391-3, J6 284391-3, J7 284391-3, J8 284391-3, J9 284391-3

Commit message: Logo updates
Parts:
- added G***: LOGO, LOGO, F.Cu at (99.9, 43.6)
- added G***: LOGO, LOGO, F.Cu at (122.4, 43.6)
